Commit message: updates for testing camera v1

File: husky_description/urdf/accessories/intel_realsense.urdf.xacro (robot description, xacro)
@@ -55,8 +55,13 @@
       </xacro:if>
     </xacro:if>
+    <!--
+      original realsense fov   h_fov:=1.5184351666666667 v_fov:=1.0122901111111111
+    -->
+    <xacro:property name="h_fov"     default="2.21657"/>
+    <xacro:property name="v_fov"     default="1.387537"/>
     <xacro:macro name="realsense_gazebo" params="
               prefix=front              model=d4
               frame:=realsense          topic:=realsense
-              h_fov:=1.5184351666666667 v_fov:=1.0122901111111111
+              h_fov:=${h_fov} v_fov:=${v_fov}
               min_range:=0.105          max_range:=8.0
               width:=640                height:=480
@@ -130,6 +135,6 @@
          frame="${prefix}_realsense_link"
          topic="${topic}"
-         h_fov="1.5184351666666667"
-         v_fov="1.0122901111111111"
+         h_fov="${h_fov}"
+         v_fov="${v_fov}"
          min_range="0.105"
          max_range="8.0"
@@ -147,6 +152,6 @@
          frame="${prefix}_realsense_link"
          topic="${topic}"
-         h_fov="1.5184351666666667"
-         v_fov="1.0122901111111111"
+         h_fov="${h_fov}"
+         v_fov="${v_fov}"
          min_range="0.105"
          max_range="8.0"
@@ -195,6 +200,6 @@
          frame="${prefix}_realsense_link"
          topic="${topic}"
-         h_fov="1.1344640137963142"
-         v_fov="0.6981317007977318"
+         h_fov="${h_fov}"
+         v_fov="${v_fov}"
          min_range="0.3"
          max_range="5.0"
@@ -213,6 +218,6 @@
          frame="${prefix}_realsense_link"
          topic="${topic}"
-         h_fov="1.5009831567151233"
-         v_fov="0.9948376736367678"
+         h_fov="${h_fov}"
+         v_fov="${v_fov}"
          min_range="0.5"
          max_range="20.0"
@@ -267,6 +272,6 @@
          frame="${prefix}_realsense_link"
          topic="${topic}"
-         h_fov="1.2217304763960306"
-         v_fov="0.9599310885968813"
+         h_fov="${h_fov}"
+         v_fov="${v_fov}"
          min_range="0.25"
          max_range="9.0"

File: husky_description/urdf/husky.urdf.xacro (robot description, xacro)
@@ -70,10 +70,10 @@
   <xacro:arg name="laser_3d_secondary_rpy"        default="$(optenv HUSKY_LASER_3D_SECONDARY_RPY 0 0 -3.14159)" />
   <!-- Realsense Camera Primary and Secondary -->
-  <xacro:arg name="realsense_enabled"             default="$(optenv HUSKY_REALSENSE_ENABLED 0)" />
+  <xacro:arg name="realsense_enabled"             default="$(optenv HUSKY_REALSENSE_ENABLED 1)" />
   <xacro:arg name="realsense_model"               default="$(optenv HUSKY_REALSENSE_MODEL d435)"/>
   <xacro:arg name="realsense_topic"               default="$(optenv HUSKY_REALSENSE_TOPIC realsense)" />
   <xacro:arg name="realsense_prefix"              default="$(optenv HUSKY_REALSENSE_PREFIX camera)" />
-  <xacro:arg name="realsense_parent"              default="$(optenv HUSKY_REALSENSE_PARENT top_plate_link)" />
-  <xacro:arg name="realsense_xyz"                 default="$(optenv HUSKY_REALSENSE_XYZ 0 0 0)" />
+  <xacro:arg name="realsense_parent"              default="$(optenv HUSKY_REALSENSE_PARENT rotation_link)" />
+  <xacro:arg name="realsense_xyz"                 default="$(optenv HUSKY_REALSENSE_XYZ 0 0 0.2)" />
   <xacro:arg name="realsense_rpy"                 default="$(optenv HUSKY_REALSENSE_RPY 0 0 0)" />
   <xacro:property name="realsense_model"          value="$(arg realsense_model)"/>
@@ -158,4 +158,33 @@
     </collision>
   </link>
+  <!-- test link for rotation -->
+  <link name="rotation_link">
+    <visual>
+      <origin xyz="0 0 0" rpy="0 0 0" />
+      <geometry>
+        <box size="0.1 0.1 0.1"/>
+      </geometry>
+    </visual>
+    <collision>
+      <origin xyz="0.1 0.1 0.1" rpy="0 0 0" />
+      <geometry>
+        <box size="0.1 0.1 0.1"/>
+      </geometry>
+    </collision>
+    <inertial>
+        <origin xyz="0 0 0" rpy="0 0 0" />
+        <mass value="0.1" />
+        <inertia
+          ixx="0.01" ixy="0.0" ixz="0.0"
+          iyy="0.01" iyz="0.0"
+          izz="0.01" />
+    </inertial>
+  </link>
+  <joint name="rotation_joint" type="continuous">
+    <origin xyz="0.5 0 0.07" rpy="0 0 0" />
+    <parent link="base_link" />
+    <child link="rotation_link" />
+		<axis xyz="0 1 0" rpy="0 0 0" />
+  </joint>
   <!-- Base footprint is on the ground under the robot -->
   <link name="base_footprint"/>
@@ -358,4 +387,13 @@
     </plugin>
   </gazebo>
+  <transmission name="rotation_trans" type="SimpleTransmission">
+    <type>transmission_interface/SimpleTransmission</type>
+    <actuator name="rotation_motor">
+      <mechanicalReduction>1</mechanicalReduction>
+    </actuator>
+    <joint name="rotation_joint">
+      <hardwareInterface>hardware_interface/EffortJointInterface</hardwareInterface>
+    </joint>
+  </transmission>
   <!-- Optional custom includes. -->
   <xacro:include filename="$(arg urdf_extras)" />
