Commit message: prismatic joint

File: husky_description/urdf/husky.urdf.xacro (robot description, xacro)
@@ -158,4 +158,49 @@
     </collision>
   </link>
+  <link name="camera_base">
+    <visual>
+      <origin xyz="0 0 0" rpy="0 0 0" />
+      <geometry>
+        <box size="0.1 0.1 0.1"/>
+      </geometry>
+    </visual>
+    <!--collision>
+      <origin xyz="0.1 0.1 0.1" rpy="0 0 0" />
+      <geometry>
+        <box size="0.1 0.1 0.1"/>
+      </geometry>
+    </collision-->
+    <inertial>
+        <origin xyz="0 0 0" rpy="0 0 0" />
+        <mass value="0.1" />
+        <inertia
+          ixx="0.01" ixy="0.0" ixz="0.0"
+          iyy="0.01" iyz="0.0"
+          izz="0.01" />
+    </inertial>
+  </link>
+ <!-- test link for camera_base -->
+  <link name="prismatic_link">
+    <visual>
+      <origin xyz="0 0 0" rpy="0 0 0" />
+      <geometry>
+        <cylinder length="0.2" radius="0.1"/>
+      </geometry>
+    </visual>
+    <!--collision>
+      <origin xyz="0.1 0.1 0.1" rpy="0 0 0" />
+      <geometry>
+        <cylinder length="0.2" radius="0.1"/>
+      </geometry>
+    </collision-->
+    <inertial>
+        <origin xyz="0 0 0" rpy="0 0 0" />
+        <mass value="0.1" />
+        <inertia
+          ixx="0.01" ixy="0.0" ixz="0.0"
+          iyy="0.01" iyz="0.0"
+          izz="0.01" />
+    </inertial>
+  </link>
   <!-- test link for rotation -->
   <link name="rotation_link">
@@ -181,7 +226,22 @@
     </inertial>
   </link>
-  <joint name="rotation_joint" type="continuous">
+  <!--camera base-->
+  <joint name="camera_base_joint" type="fixed">
     <origin xyz="0.5 0 0.07" rpy="0 0 0" />
     <parent link="base_link" />
+    <child link="camera_base" />
+  </joint>
+  <!--camera prismatic-->
+  <joint name="prismatic_joint" type="prismatic">
+    <origin xyz="0.0 0 0.2" rpy="0 0 0" />
+    <parent link="camera_base" />
+    <child link="prismatic_link" />
+		<axis xyz="0 0 1" rpy="0 0 0" />
+    <limit lower="-1" upper="1" effort="23000" velocity="0.1"/>
+  </joint>
+  <!--camera rotation joint-->
+  <joint name="rotation_joint" type="continuous">
+    <origin xyz="0 0 0.0" rpy="0 0 0" />
+    <parent link="prismatic_link" />
     <child link="rotation_link" />
 		<axis xyz="0 1 0" rpy="0 0 0" />
@@ -387,4 +447,14 @@
     </plugin>
   </gazebo>
+  <transmission name="prismatic_trans" type="SimpleTransmission">
+    <type>transmission_interface/SimpleTransmission</type>
+    <actuator name="prismatic_motor">
+      <mechanicalReduction>1</mechanicalReduction>
+      <hardwareInterface>hardware_interface/EffortJointInterface</hardwareInterface>
+    </actuator>
+    <joint name="prismatic_joint">
+      <hardwareInterface>hardware_interface/EffortJointInterface</hardwareInterface>
+    </joint>
+  </transmission>
   <transmission name="rotation_trans" type="SimpleTransmission">
     <type>transmission_interface/SimpleTransmission</type>
